Commit message: updates

File: Workshop_4/slam_dunk.urdf.xacro (robot description, xacro)
@@ -2,8 +2,9 @@
 <robot xmlns:xacro="http://ros.org/wiki/xacro"
        name="slam_dunk" >
-	<!-- THE ROBOT -->
+	<!-- the robot's static environment -->
 	<link name="world" />
-	<!-- UR from ROS-i repos -->
+	<!-- the UR5 Robot -->
 	<xacro:include filename="$(find ur_description)/urdf/ur5.urdf.xacro" />
+	<xacro:ur5_robot prefix="ur5_" joint_limited="true" />
 	<joint name="world_joint" type="fixed">
 		<parent link="world" />
@@ -11,9 +12,3 @@
 		<origin xyz="0.0 0.0 0.0" rpy="0.0 0.0 0.0" />
 	</joint>
-	<xacro:ur5_robot prefix="ur5_" joint_limited="true" />
-	<!-- Robotiq from Beta Robots fork-->
-	<!-- <xacro:include filename="$(find robotiq_85_description)/urdf/robotiq_85_gripper.urdf.xacro" />
-	<xacro:robotiq_85_gripper prefix="simple_gripper_" parent="simple_arm_tool0">
-		<origin xyz="0 0 0" rpy="${pi/2} -${pi/2} 0" />
-	</xacro:robotiq_85_gripper> -->
 </robot>
